File: HVPSU-Projects/HVTest/CW-Chain.sch (KiCad schematic (older format))
At the start: 113 parts, among them J2 SMA, J3 UFL-CONN, J4 RF_SHIELD_TWO_PIECES, P13 CONN_01X02, P17 CONN_01X01, Q1 NMOS-DMG3420U, U14 MAX9634

Commit message: latest
Parts:
- GND1, P17, ST1, ST10, ST11, ST12, ST2, ST3, ST4, ST5, ST6, ST7, ST8, ST9: symbol conn:CONN_01X01 -> HVTest-rescue:CONN_01X01-conn
- OUT1: symbol conn:TEST_1P -> HVTest-rescue:TEST_1P-conn
- P13: symbol conn:CONN_01X02 -> HVTest-rescue:CONN_01X02-conn
Changed lines of the file:
@@
 HVR
 $Comp
-L conn:CONN_01X01 ST12
+L HVTest-rescue:CONN_01X01-conn ST12
 U 1 1 5856B25C
 P 10600 4750
@@
 $EndComp
 $Comp
-L conn:CONN_01X01 ST11
+L HVTest-rescue:CONN_01X01-conn ST11
 U 1 1 5856C812
 P 9200 4750
@@
 $EndComp
 $Comp
-L conn:CONN_01X01 ST10
+L HVTest-rescue:CONN_01X01-conn ST10
 U 1 1 5856D17C
 P 8800 4750
@@
 $EndComp
 $Comp
-L conn:CONN_01X01 ST9
+L HVTest-rescue:CONN_01X01-conn ST9
 U 1 1 5856D2A9
 P 8100 4750
@@
 $EndComp
 $Comp
-L conn:CONN_01X01 ST8
+L HVTest-rescue:CONN_01X01-conn ST8
 U 1 1 5856D3E9
 P 7700 4750
@@
 $EndComp
 $Comp
-L conn:CONN_01X01 ST7
+L HVTest-rescue:CONN_01X01-conn ST7
 U 1 1 5856D51C
 P 7000 4750
@@
 $EndComp
 $Comp
-L conn:CONN_01X01 ST6
+L HVTest-rescue:CONN_01X01-conn ST6
 U 1 1 5856D660
 P 6600 4750
@@
 $EndComp
 $Comp
-L conn:CONN_01X01 ST5
+L HVTest-rescue:CONN_01X01-conn ST5
 U 1 1 5856D857
 P 5900 4750
@@
 $EndComp
 $Comp
-L conn:CONN_01X01 ST4
+L HVTest-rescue:CONN_01X01-conn ST4
 U 1 1 5856D99F
 P 5500 4750
@@
 $EndComp
 $Comp
-L conn:CONN_01X01 ST3
+L HVTest-rescue:CONN_01X01-conn ST3
 U 1 1 5856DAE2
 P 4800 4750
@@
 $EndComp
 $Comp
-L conn:CONN_01X01 ST2
+L HVTest-rescue:CONN_01X01-conn ST2
 U 1 1 5856DC34
 P 4400 4750
@@
 $EndComp
 $Comp
-L conn:CONN_01X01 ST1
+L HVTest-rescue:CONN_01X01-conn ST1
 U 1 1 5856DD7D
 P 3700 4750
@@
 	2250 3700 2250 3450
 $Comp
-L conn:TEST_1P OUT1
+L HVTest-rescue:TEST_1P-conn OUT1
 U 1 1 5855312C
 P 2200 5900
@@
 Connection ~ 2200 6050
 $Comp
-L conn:CONN_01X01 GND1
+L HVTest-rescue:CONN_01X01-conn GND1
 U 1 1 5855504B
 P 3050 4750
@@
 	3050 4400 3050 4550
 $Comp
-L conn:CONN_01X02 P13
+L HVTest-rescue:CONN_01X02-conn P13
 U 1 1 5855F11B
 P 1200 3450
@@
 Optional
 $Comp
-L conn:CONN_01X01 P17
+L HVTest-rescue:CONN_01X01-conn P17
 U 1 1 5889C947
 P 10450 4100
