File: HVPSU-Projects/HVTest/CheetahSocket.sch (KiCad schematic (older format))
At the start: 12 parts, among them J5 HIROSE-DF12, P14 CONN_01X03, P23 CONN_01X01, P24 CONN_01X01, P25 CONN_01X02, U11 TLP293-4

Commit message: latest
Parts:
- P14: symbol conn:CONN_01X03 -> HVTest-rescue:CONN_01X03-conn
- P23, P24: symbol conn:CONN_01X01 -> HVTest-rescue:CONN_01X01-conn
- P25: symbol conn:CONN_01X02 -> HVTest-rescue:CONN_01X02-conn
Changed lines of the file:
@@
 NoConn ~ 7500 3350
 $Comp
-L conn:CONN_01X03 P14
+L HVTest-rescue:CONN_01X03-conn P14
 U 1 1 5879274E
 P 6050 4750
@@
 Connection ~ 6650 4050
 $Comp
-L conn:CONN_01X01 P23
+L HVTest-rescue:CONN_01X01-conn P23
 U 1 1 5891701B
 P 6500 4750
@@
 $EndComp
 $Comp
-L conn:CONN_01X01 P24
+L HVTest-rescue:CONN_01X01-conn P24
 U 1 1 589170B8
 P 6650 4750
@@
 	6650 5000 6500 5000
 $Comp
-L conn:CONN_01X02 P25
+L HVTest-rescue:CONN_01X02-conn P25
 U 1 1 5893B04C
 P 7150 2750
