File: HVPSU-Projects/HVTest/Comms.sch (KiCad schematic (older format))
At the start: 15 parts, among them J1 USB-MICRO-B, P19 CONN_01X02, U1 NUF2101MT1G, U2 FT230X

Commit message: latest
Parts:
- P19: symbol conn:CONN_01X02 -> HVTest-rescue:CONN_01X02-conn
Changed lines of the file:
@@
 Connection ~ 2250 4900
 $Comp
-L conn:CONN_01X02 P19
+L HVTest-rescue:CONN_01X02-conn P19
 U 1 1 5889E948
 P 7300 3800
