File: HVPSU-Projects/HVTest/DACs.sch (KiCad schematic (older format))
At the start: 6 parts, among them U5 MAX5531, U6 MCP4912

Commit message: latest
Parts:
- W1: symbol conn:TEST_1P -> HVTest-rescue:TEST_1P-conn
Changed lines of the file:
@@
 Connection ~ 5500 3000
 $Comp
-L conn:TEST_1P W1
+L HVTest-rescue:TEST_1P-conn W1
 U 1 1 5884B643
 P 6700 3600
