File: HVPSU-Projects/HVTest/HVMeasurement.sch (KiCad schematic (older format))
At the start: 13 parts, among them P15 CONN_01X02, P18 CONN_01X01, U12 LTC2050, U13 LTC2451

Commit message: latest
Parts:
- P15: symbol conn:CONN_01X02 -> HVTest-rescue:CONN_01X02-conn
- P18: symbol conn:CONN_01X01 -> HVTest-rescue:CONN_01X01-conn
Changed lines of the file:
@@
 $EndComp
 $Comp
-L conn:CONN_01X02 P15
+L HVTest-rescue:CONN_01X02-conn P15
 U 1 1 587A31B3
 P 6350 4100
@@
 Connect 100G Res
 $Comp
-L conn:CONN_01X01 P18
+L HVTest-rescue:CONN_01X01-conn P18
 U 1 1 5889AE54
 P 4050 3050
+AR Path="/5889AE54" Ref="P18"  Part="1"
+AR Path="/5879B204/5889AE54" Ref="P18"  Part="1"
 F 0 "P18" H 4050 3150 50  0000 C CNN
 F 1 "CONN_01X01" V 4150 3050 50  0000 C CNN
