File: HVPSU-Projects/HVTest/Power.sch (KiCad schematic (older format))
At the start: 12 parts, among them P1 CONN_01X02, P2 CONN_01X03, P3 CONN_01X03, P4 CONN_01X03, P5 CONN_01X01, P6 CONN_01X01, P7 CONN_01X01, U4 MCP1700t-3302E/TT

Commit message: latest
Parts:
- P1: symbol conn:CONN_01X02 -> HVTest-rescue:CONN_01X02-conn
- P2, P3, P4: symbol conn:CONN_01X03 -> HVTest-rescue:CONN_01X03-conn
- P5, P6, P7: symbol conn:CONN_01X01 -> HVTest-rescue:CONN_01X01-conn
Changed lines of the file:
@@
 	6650 4000 6650 3850
 $Comp
-L conn:CONN_01X03 P2
+L HVTest-rescue:CONN_01X03-conn P2
 U 1 1 5853E594
 P 9450 3900
@@
 $EndComp
 $Comp
-L conn:CONN_01X01 P5
+L HVTest-rescue:CONN_01X01-conn P5
 U 1 1 5853E987
 P 9550 3900
@@
 $EndComp
 $Comp
-L conn:CONN_01X03 P3
+L HVTest-rescue:CONN_01X03-conn P3
 U 1 1 5853F361
 P 9450 4750
@@
 $EndComp
 $Comp
-L conn:CONN_01X01 P6
+L HVTest-rescue:CONN_01X01-conn P6
 U 1 1 5853F3A5
 P 9550 4750
@@
 	9250 4650 9150 4650
 $Comp
-L conn:CONN_01X03 P4
+L HVTest-rescue:CONN_01X03-conn P4
 U 1 1 5853F666
 P 9450 5600
@@
 $EndComp
 $Comp
-L conn:CONN_01X01 P7
+L HVTest-rescue:CONN_01X01-conn P7
 U 1 1 5853F6AC
 P 9550 5600
@@
 CW Chain Supply
 $Comp
-L conn:CONN_01X02 P1
+L HVTest-rescue:CONN_01X02-conn P1
 U 1 1 585433B4
 P 7400 4000
