File: HVPSU-Projects/HVTest/SwitchIC.sch (KiCad schematic (older format))
At the start: 23 parts, among them P16 CONN_01X02, P21 CONN_01X03, P22 CONN_01X02, P8 CONN_01X02, U7 switch_ic4/5

Commit message: latest
Parts:
- P16, P22, P8: symbol conn:CONN_01X02 -> HVTest-rescue:CONN_01X02-conn
- P21: symbol conn:CONN_01X03 -> HVTest-rescue:CONN_01X03-conn
- RST1: symbol conn:TEST_1P -> HVTest-rescue:TEST_1P-conn
Changed lines of the file:
@@
 Connects to 50k digipot\nChannel 1
 $Comp
-L conn:CONN_01X02 P8
+L HVTest-rescue:CONN_01X02-conn P8
 U 1 1 585659D2
 P 4300 4100
@@
 $EndComp
 $Comp
-L conn:CONN_01X03 P21
+L HVTest-rescue:CONN_01X03-conn P21
 U 1 1 588003E0
 P 3600 3300
@@
 $EndComp
 $Comp
-L conn:TEST_1P RST1
+L HVTest-rescue:TEST_1P-conn RST1
 U 1 1 58803EC0
 P 8300 3750
@@
 MSB
 $Comp
-L conn:CONN_01X02 P22
+L HVTest-rescue:CONN_01X02-conn P22
 U 1 1 5884C862
 P 4900 4600
@@
 $EndComp
 $Comp
-L conn:CONN_01X02 P16
+L HVTest-rescue:CONN_01X02-conn P16
 U 1 1 5887DD22
 P 7150 5000
