File: HVPSU-Projects/HVTest/Switches-Digipots.sch (KiCad schematic (older format))
At the start: 16 parts, among them P10 CONN_01X02, P11 CONN_01X02, P12 CONN_01X02, P9 CONN_01X02, U10 MCP4651T, U8 MAX4704, U9 MAX4704

Commit message: latest
Parts:
- P10, P11, P12, P9: symbol conn:CONN_01X02 -> HVTest-rescue:CONN_01X02-conn
Changed lines of the file:
@@
 Analog switch to select\npulse width timing cap
 $Comp
-L conn:CONN_01X02 P11
+L HVTest-rescue:CONN_01X02-conn P11
 U 1 1 58539293
 P 9000 4600
@@
 $EndComp
 $Comp
-L conn:CONN_01X02 P12
+L HVTest-rescue:CONN_01X02-conn P12
 U 1 1 585395C9
 P 9450 4350
@@
 Connection ~ 8650 4550
 $Comp
-L conn:CONN_01X02 P9
+L HVTest-rescue:CONN_01X02-conn P9
 U 1 1 5853AA87
 P 3850 1350
@@
 $EndComp
 $Comp
-L conn:CONN_01X02 P10
+L HVTest-rescue:CONN_01X02-conn P10
 U 1 1 5853BB24
 P 3750 4600
